File: anavi-gardening-controller.kicad_pcb (KiCad board)
At the start: 2 copper layers, 57.7 x 47.2 mm, 20 parts, among them J1 Conn_01x04_Female, J2 Conn_01x04_Female, J3 Conn_01x04_Female, J4 Conn_01x04_Female, J5 Conn_02x04_Odd_Even, U1 MOUDLE-SEEEDUINO-XIAO-ESP32C3, U2 DS18B20

Commit message: Update to KiCad 8
Update the project to KiCad version 8. Tested with 8.0.5 on
Ubuntu 2024.04 LTS.

Signed-off-by: Leon Anavi <leon@anavi.org>
Parts:
- LED1: value LED -> KP-3216EC
